File: h-drivers.sch (KiCad schematic (older format))
At the start: 36 parts

Commit message: Added Green LED for signalling VBB
Parts:
- removed R?: R, symbol Device:R
- added D?: GREEN, symbol Device:LED
- added Q?: 2N7002, Package_TO_SOT_SMD:SOT-23, symbol Transistor_FET:2N7002
- added R?: 4.7k, symbol Device:R
- added R?: 110, symbol Device:R
- added R?: 10k, symbol Device:R
Connections:
- wire segments 149 -> 159
Other:
- moved on the sheet: C?, D?, L?, R?, RV?, U?
