File: plc-utility-board.kicad_pcb (KiCad board)
At the start: 2 copper layers, 127 parts, among them J1 Screw_Terminal_01x02, J10 Screw_Terminal_01x03, J11 Screw_Terminal_01x02, J2 Screw_Terminal_01x08, J3 Screw_Terminal_01x04, J4 Screw_Terminal_01x08, J5 TerminalBlock_02x04, J6 Conn_01x03_Male, J7 Conn_01x03_Male, J8 Screw_Terminal_01x03, J9 Screw_Terminal_01x02, Q1 2N7002, Q10 2N7002, Q11 2N7002, Q12 2N7002, Q13 2N7002, Q14 2N7002, Q15 2N7002, Q16 2N7002, Q2 2N7002, Q3 BC327, Q4 BC327, Q5 2N7002, Q6 2N7002, Q7 BC327, Q8 BC327, Q9 2N7002, U1 MAX15062A, U2 A8498, U3 A3950SLP-T, U4 A8498, U5 A3950SLP-T

Commit message: Added power supply section to PCB. Added missing components footprints.
Parts:
- removed C21: 0.1uF 50V, Capacitor_SMD:C_0805_2012Metric_Pad1.15x1.40mm_HandSolder
- added D8: RED, LED_SMD:LED_0603_1608Metric_Pad1.05x0.95mm_HandSolder, F.Cu at (241.3, 162.6)
- C1: value 1uF -> 22uF 50V; footprint Capacitor_SMD:C_0805_2012Metric_Pad1.15x1.40mm_HandSolder -> Capacitor_THT:CP_Radial_D5.0mm_P2.00mm
- C10, C19: value 100uF -> 0.22uF 25V; footprint Capacitor_SMD:CP_Elec_8x10.5 -> Capacitor_SMD:C_0603_1608Metric_Pad1.05x0.95mm_HandSolder
- C11, C20: value 0.22uF 25V -> 0.1uF 50V; footprint Capacitor_SMD:C_0603_1608Metric_Pad1.05x0.95mm_HandSolder -> Capacitor_SMD:C_0805_2012Metric_Pad1.15x1.40mm_HandSolder
- C12: value 0.1uF 50V -> 0.01uF; footprint Capacitor_SMD:C_0805_2012Metric_Pad1.15x1.40mm_HandSolder -> Capacitor_SMD:C_0603_1608Metric_Pad1.05x0.95mm_HandSolder
- C13, C4: value 0.01uF -> 82uF; footprint Capacitor_SMD:C_0603_1608Metric_Pad1.05x0.95mm_HandSolder -> Capacitor_SMD:CP_Elec_6.3x5.8
- C14, C5: value 82uF -> 330uF; footprint Capacitor_SMD:CP_Elec_6.3x5.8 -> Capacitor_SMD:CP_Elec_6.3x7.7
- C15, C6: value 330uF -> 0.1uF; footprint Capacitor_SMD:CP_Elec_6.3x7.7 -> Capacitor_SMD:C_0805_2012Metric_Pad1.15x1.40mm_HandSolder
- C16, C7: value 0.1uF -> 0.1uF 50V
- C18, C9: value 0.1uF 50V -> 100uF; footprint Capacitor_SMD:C_0805_2012Metric_Pad1.15x1.40mm_HandSolder -> Capacitor_SMD:CP_Elec_8x10.5
- C2: value 1uF -> 220uF 25V; footprint Capacitor_SMD:C_0805_2012Metric_Pad1.15x1.40mm_HandSolder -> Capacitor_THT:CP_Radial_D6.3mm_P2.50mm
- C3: value 10uF -> 0.01uF; footprint Capacitor_SMD:C_0805_2012Metric_Pad1.15x1.40mm_HandSolder -> Capacitor_SMD:C_0603_1608Metric_Pad1.05x0.95mm_HandSolder; moved to B.Cu
- D1: value SSC53L -> SB530; footprint Diode_SMD:D_SMC_Handsoldering -> Diode_THT:D_DO-201_P3.81mm_Vertical_AnodeUp
- D2: value B330 -> SL04-E3-08; footprint Diode_SMD:D_SMA_Handsoldering -> Diode_SMD:D_1210_3225Metric_Pad1.42x2.65mm_HandSolder
- D3, D6: value GREEN -> B330; footprint LED_SMD:LED_0603_1608Metric_Pad1.05x0.95mm_HandSolder -> Diode_SMD:D_SMA
- D4, D7: value RED -> GREEN
- D5: value B330 -> RED; footprint Diode_SMD:D_SMA_Handsoldering -> LED_SMD:LED_0603_1608Metric_Pad1.05x0.95mm_HandSolder
- L1: value 33uH -> SRF1260-100M; footprint Inductor_SMD:L_Coilcraft_LPS4018 -> IND_SRF1260-100M
- Q1, Q10, Q11, Q12, Q13, Q14, Q15, Q16, Q2, Q5, Q6, Q9: footprint Package_TO_SOT_SMD:SOT-23 -> Package_TO_SOT_SMD:SOT-23_Handsoldering
- U1: value MAX15062A -> LM2574M-3.3; footprint Package_DFN_QFN:DFN-8-1EP_2x2mm_P0.5mm_EP0.9x1.5mm -> Package_SO:SOIC-14W_7.5x9.0mm_P1.27mm
- moved D1 235.4 mm to (106.7, 77.2), turned to 270 degrees
- moved C1 233.7 mm to (115.1, 89.2), turned to 180 degrees
- moved U1 228.8 mm to (116.3, 79.2), turned to 270 degrees
- moved L1 221.4 mm to (128.8, 83.4), turned to 180 degrees
- moved C2 199.3 mm to (139.6, 79.1), turned to 270 degrees
- moved J1 180.6 mm to (106.7, 90.9), turned to 90 degrees
- moved D2 147.0 mm to (119.6, 89.2), turned to 270 degrees
- moved U2 135.1 mm to (154.3, 90.8)
- moved C3 129.2 mm to (205.1, 139.7)
- moved J10 125.2 mm to (181.6, 120.7), turned to 180 degrees
- moved J9 113.0 mm to (176.8, 51.3)
- moved J11 111.7 mm to (197.0, 54.8)
- moved Q8 110.1 mm to (208.9, 7.42), turned to 270 degrees
- moved Q7 109.0 mm to (196.2, 7.42), turned to 270 degrees
- moved J3 101.2 mm to (227.3, 41.9)
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Connections:
- C10 pad 1: /Motor1 driver/VBB -> GND
- C10 pad 2: GND -> Net-(C10-Pad2)
- C11 pad 1: GND -> Net-(C11-Pad1)
- C13 pad 1: Net-(C13-Pad1) -> /Motor1 supply/24V
- C13 pad 2: Net-(C13-Pad2) -> GND
- C14 pad 1: /Motor1 supply/24V -> /Motor2 driver/VBB
- C15 pad 1: /Motor2 driver/VBB -> GND
- C15 pad 2: GND -> /Motor1 supply/24V
- C16 pad 1: GND -> /Motor2 driver/VBB
- C16 pad 2: /Motor1 supply/24V -> GND
- C17 pad 2: GND -> Net-(C17-Pad2)
- C18 pad 2: Net-(C18-Pad2) -> GND
- C19 pad 1: /Motor2 driver/VBB -> GND
- C19 pad 2: GND -> Net-(C19-Pad2)
- C2 pad 1: Net-(C2-Pad1) -> /Motor1 3V3 <- PLC/3V3
- C20 pad 1: GND -> Net-(C20-Pad1)
- C3 pad 1: /Motor1 3V3 <- PLC/3V3 -> Net-(C3-Pad1)
- C3 pad 2: GND -> Net-(C3-Pad2)
- C4 pad 1: Net-(C4-Pad1) -> /Motor1 supply/24V
- C4 pad 2: Net-(C4-Pad2) -> GND
- C5 pad 1: /Motor1 supply/24V -> /Motor1 driver/VBB
- C6 pad 1: /Motor1 driver/VBB -> GND
- C6 pad 2: GND -> /Motor1 supply/24V
- C7 pad 1: GND -> /Motor1 driver/VBB
- C7 pad 2: /Motor1 supply/24V -> GND
- C8 pad 2: GND -> Net-(C8-Pad2)
- C9 pad 2: Net-(C9-Pad2) -> GND
- D2 pad 1: Net-(C4-Pad2) -> Net-(D2-Pad1)
- D3 pad 1: Net-(D3-Pad1) -> Net-(C3-Pad2)
- D3 pad 2: Net-(D3-Pad2) -> GND
- D4 pad 2: /Motor1 3V3 <- PLC/3V3 -> Net-(D4-Pad2)
- D5 pad 1: Net-(C13-Pad2) -> Net-(D5-Pad1)
- D5 pad 2: GND -> /Motor1 3V3 <- PLC/3V3
- D6 pad 1: Net-(D6-Pad1) -> Net-(C12-Pad2)
- D6 pad 2: Net-(D6-Pad2) -> GND
- D7 pad 2: /Motor1 3V3 <- PLC/3V3 -> Net-(D7-Pad2)
- J1 pad 1: /Power section/VIN -> GND
- J1 pad 2: GND -> /Power section/VIN
- J3 pad 1: /ttl-to-plc/IN1 -> /ttl-to-plc/IN4
- J3 pad 2: /ttl-to-plc/IN2 -> /ttl-to-plc/IN3
- J3 pad 3: /ttl-to-plc/IN3 -> /ttl-to-plc/IN2
- J3 pad 4: /ttl-to-plc/IN4 -> /ttl-to-plc/IN1
- L1 pad 1: Net-(L1-Pad1) -> Net-(D2-Pad1)
- L1 pad 2: /Motor1 3V3 <- PLC/3V3 -> Net-(D2-Pad1)
- L2 pad 1: Net-(C4-Pad2) -> Net-(C3-Pad2)
- L3 pad 1: Net-(C13-Pad2) -> Net-(C12-Pad2)
- Q13 pad 3: Net-(D6-Pad1) -> Net-(D7-Pad1)
- Q9 pad 3: Net-(D3-Pad1) -> Net-(D4-Pad1)
- R26 pad 2: Net-(D3-Pad2) -> Net-(D4-Pad2)
- R28 pad 1: Net-(D4-Pad1) -> Net-(D5-Pad1)
- R43 pad 2: Net-(D6-Pad2) -> Net-(D7-Pad2)
- R45 pad 1: Net-(D7-Pad1) -> Net-(D8-Pad1)
- U1 pad 1: /Motor1 supply/24V -> (no net)
- U1 pad 2: /Motor1 supply/24V -> (no net)
- U1 pad 3: Net-(C2-Pad1) -> /Motor1 3V3 <- PLC/3V3
- U1 pad 4: /Motor1 3V3 <- PLC/3V3 -> GND
- U1 pad 5: Net-(U1-Pad5) -> GND
- U1 pad 6: Net-(U1-Pad6) -> GND
- U1 pad 7: GND -> (no net)
- U1 pad 8: Net-(L1-Pad1) -> (no net)
- U2 pad 1: Net-(C4-Pad1) -> Net-(C3-Pad1)
- U2 pad 7: Net-(C4-Pad2) -> Net-(C3-Pad2)
- U3 pad 11: Net-(C12-Pad1) -> Net-(C11-Pad1)
- U3 pad 12: Net-(C12-Pad2) -> Net-(C11-Pad2)
- U3 pad 14: Net-(C9-Pad2) -> Net-(C8-Pad2)
- U3 pad 15: Net-(C11-Pad2) -> Net-(C10-Pad2)
- U4 pad 1: Net-(C13-Pad1) -> Net-(C12-Pad1)
- U4 pad 7: Net-(C13-Pad2) -> Net-(C12-Pad2)
- U5 pad 11: Net-(C21-Pad1) -> Net-(C20-Pad1)
- U5 pad 12: Net-(C21-Pad2) -> Net-(C20-Pad2)
- U5 pad 14: Net-(C18-Pad2) -> Net-(C17-Pad2)
- U5 pad 15: Net-(C20-Pad2) -> Net-(C19-Pad2)
Routing:
- net /plc-to-ttl/OUT4: track 32.8 -> 0.00 mm
- net /plc-to-ttl/OUT8: track 32.8 -> 0.00 mm
- net /plc-to-ttl/OUT6: track 32.8 -> 0.00 mm
- net /plc-to-ttl/OUT2: track 32.8 -> 0.00 mm
- net /plc-to-ttl/IN7: track 31.5 -> 0.00 mm
- net /plc-to-ttl/IN5: track 31.5 -> 0.00 mm
- net /plc-to-ttl/IN3: track 31.5 -> 0.00 mm
- net /plc-to-ttl/IN1: track 31.5 -> 0.00 mm
- net /Motor1 3V3 <- PLC/3V3: track 0.00 -> 24.6 mm
- net /Motor1 supply/24V: track 0.00 -> 18.4 mm
- net /plc-to-ttl/OUT7: track 17.8 -> 0.00 mm
- net /plc-to-ttl/OUT5: track 17.8 -> 0.00 mm
- net /plc-to-ttl/OUT3: track 17.8 -> 0.00 mm
- net /plc-to-ttl/OUT1: track 17.8 -> 0.00 mm
- net /plc-to-ttl/IN8: track 16.5 -> 0.00 mm
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Other:
- net class Default: clearance 0.2 -> 0.254
- rule trace_clearance: 0.2 -> 0.254

Commit message: PCB creation, improvements of power supply section
Parts:
- C3: moved to F.Cu
- L1: footprint IND_SRF1260-100M -> SRF1260-100M:IND_SRF1260-100M
- Q10, Q11, Q12, Q14, Q15, Q16: footprint Package_TO_SOT_SMD:SOT-23_Handsoldering -> Package_TO_SOT_SMD:SuperSOT-3
- R21, R22, R38: footprint Resistor_SMD:R_0805_2012Metric_Pad1.15x1.40mm_HandSolder -> Resistor_SMD:R_0603_1608Metric_Pad1.05x0.95mm_HandSolder
- R23: value 16k -> 10k; footprint Resistor_SMD:R_0805_2012Metric_Pad1.15x1.40mm_HandSolder -> Resistor_SMD:R_0603_1608Metric_Pad1.05x0.95mm_HandSolder
- R24, R29, R32, R35, R41, R46, R49, R52: footprint Resistor_SMD:R_1206_3216Metric_Pad1.42x1.75mm_HandSolder -> Resistor_SMD:R_0805_2012Metric_Pad1.15x1.40mm_HandSolder
- R40: value 16k -> 10k
- RV1, RV10: value 47k -> 50k; footprint Potentiometer_THT:Potentiometer_Bourns_3386P_Vertical -> Potentiometer_THT:Potentiometer_Vishay_T73XX_Horizontal
- moved U4 210.6 mm to (168.9, 35.6)
- moved U3 198.0 mm to (147.3, 98.6), turned to 180 degrees
- moved J6 169.6 mm to (155.4, 104.1), turned to 270 degrees
- moved Q12 148.3 mm to (145.3, 108.8), turned to 180 degrees
- moved R36 143.9 mm to (143.9, 113.0), turned to 270 degrees
- moved R37 142.0 mm to (148.9, 108.9), turned to 270 degrees
- moved R35 138.0 mm to (146.4, 113.0), turned to 270 degrees
- moved R34 137.0 mm to (156.2, 108.9), turned to 270 degrees
- moved Q10 136.7 mm to (159.8, 108.9), turned to 180 degrees
- moved D3 135.8 mm to (159.0, 74.9), turned to 180 degrees
- moved Q11 132.8 mm to (152.6, 108.9), turned to 180 degrees
- moved R32 132.0 mm to (153.7, 113.0), turned to 270 degrees
- moved R33 131.6 mm to (151.1, 113.0), turned to 270 degrees
- moved R21 130.9 mm to (144.8, 82.5)
- moved RV1 130.7 mm to (150.9, 85.1), turned to 270 degrees
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Connections:
- J6 pad 1: /Motor1 driver/MODE -> /Motor1 driver/ENABLE
- J6 pad 3: /Motor1 driver/ENABLE -> /Motor1 driver/MODE
- Q10 pad 2: /Motor1 driver/MODE -> /Motor1 driver/ENABLE
- Q12 pad 2: /Motor1 driver/ENABLE -> /Motor1 driver/MODE
- R31 pad 1: /Motor1 driver/MODE -> /Motor1 driver/ENABLE
- R37 pad 1: /Motor1 driver/ENABLE -> /Motor1 driver/MODE
- RV1 pad 3: GND -> Net-(RV1-Pad3)
- RV10 pad 3: GND -> Net-(RV10-Pad3)
Routing:
- net /Motor1 supply/24V: track 18.4 -> 0.00 mm
- net /Motor1 3V3 <- PLC/3V3: track 24.6 -> 10.9 mm
- net Net-(D2-Pad1): track 16.1 -> 10.6 mm
- net /Power section/VIN: track 4.83 -> 0.00 mm

Commit message: Further work at PCB
Parts:
- C1: footprint Capacitor_THT:CP_Radial_D5.0mm_P2.00mm -> Capacitor_SMD:CP_Elec_5x5.8
- D1: footprint Diode_THT:D_DO-201_P3.81mm_Vertical_AnodeUp -> PTVS3V3P1UP:SOD128
- D2: footprint Diode_SMD:D_1210_3225Metric_Pad1.42x2.65mm_HandSolder -> Diode_SMD:D_SOD-123F
- R1, R10, R11, R12, R13, R14, R17, R18, R19, R2, R20, R24, R25, R26, R27, R28, R29, R3, R30, R31, R32, R33, R34, R35, R36, R37, R39, R4, R40, R41, R42, R43, R44, R45, R46, R47, R48, R49, R50, R51, R52, R53, R54, R7, R8, R9: footprint Resistor_SMD:R_0805_2012Metric_Pad1.15x1.40mm_HandSolder -> Resistor_SMD:R_0603_1608Metric_Pad1.05x0.95mm_HandSolder
- R15, R16, R5, R6: footprint Resistor_SMD:R_1206_3216Metric_Pad1.42x1.75mm_HandSolder -> Resistor_SMD:R_0805_2012Metric_Pad1.15x1.40mm_HandSolder
- moved C3 2.69 mm to (154.3, 79.1)
- moved L2 2.69 mm to (162.9, 86.2)
- moved R21 2.69 mm to (146.7, 84.5)
- moved R23 2.69 mm to (154.3, 82.7)
- moved RV1 2.69 mm to (152.8, 87.0)
- moved U2 2.69 mm to (149.2, 80.6)
- moved D3 2.69 mm to (160.9, 76.8)
- moved R22 2.69 mm to (151.0, 84.5)
- moved J4 2.54 mm to (105.4, 69.2)
- moved C1 2.22 mm to (117.1, 90.3)
- moved D1 2.19 mm to (108.8, 90.4), turned to 180 degrees
- moved J9 2.01 mm to (153.0, 69.2)
- moved J1 1.27 mm to (106.7, 78.7)
- moved D2 0.13 mm to (128.0, 91.9)
- moved C2 0.06 mm to (137.8, 78.7)
Connections:
- RV1 pad 1: Net-(R23-Pad2) -> Net-(RV1-Pad1)
- RV1 pad 2: Net-(R22-Pad2) -> Net-(R23-Pad2)
- RV1 pad 3: Net-(RV1-Pad3) -> Net-(R22-Pad2)
- RV10 pad 1: Net-(R40-Pad2) -> Net-(RV10-Pad1)
- RV10 pad 2: Net-(R39-Pad2) -> Net-(R40-Pad2)
- RV10 pad 3: Net-(RV10-Pad3) -> Net-(R39-Pad2)
Routing:
- net Net-(D2-Pad1): track 10.6 -> 18.8 mm
- net /Motor1 3V3 <- PLC/3V3: track 10.9 -> 14.4 mm

Commit message: Changed Motor Controller to DRV8840, removed pre-motor power section. Replaced PNP transistors in logic level shifters with P-MOSFET units
Parts:
- removed C15: 0.1uF, Capacitor_SMD:C_0805_2012Metric_Pad1.15x1.40mm_HandSolder
- removed C16, C17, C20: 0.1uF 50V, Capacitor_SMD:C_0805_2012Metric_Pad1.15x1.40mm_HandSolder
- removed C18: 100uF, Capacitor_SMD:CP_Elec_8x10.5
- removed C19: 0.22uF 25V, Capacitor_SMD:C_0603_1608Metric_Pad1.05x0.95mm_HandSolder
- removed D5, D8: RED, LED_SMD:LED_0603_1608Metric_Pad1.05x0.95mm_HandSolder
- removed D6: B330, Diode_SMD:D_SMA
- removed D7: GREEN, LED_SMD:LED_0603_1608Metric_Pad1.05x0.95mm_HandSolder
- removed L1: SRF1260-100M, SRF1260-100M:IND_SRF1260-100M
- removed L2, L3: 47uH, Inductor_SMD:L_Bourns_SRP1245A
- removed R43: 110, Resistor_SMD:R_0603_1608Metric_Pad1.05x0.95mm_HandSolder
- removed R44: 5k, Resistor_SMD:R_0603_1608Metric_Pad1.05x0.95mm_HandSolder
- removed R45: 220, Resistor_SMD:R_0603_1608Metric_Pad1.05x0.95mm_HandSolder
- removed U4: A8498, Package_SO:SOIC-8-1EP_3.9x4.9mm_P1.27mm_EP2.35x2.35mm
- removed U5: A3950SLP-T, Package_SO:HTSSOP-16-1EP_4.4x5mm_P0.65mm_EP3.4x5mm_Mask3x3mm_ThermalVias
- added J12: Screw_Terminal_01x04, TerminalBlock_Phoenix:TerminalBlock_Phoenix_MKDS-1,5-4-5.08_1x04_P5.08mm_Horizontal, F.Cu at (107.8, 101.3)
- added SW1: SW_Push, Button_Switch_SMD:SW_SPST_KMR2, F.Cu at (267.3, 94.5)
- added SW2: SW_Push, Button_Switch_SMD:SW_SPST_KMR2, F.Cu at (139.4, 105.0)
- added SW3: SW_Push, Button_Switch_SMD:SW_SPST_KMR2, F.Cu at (278.4, 94.5)
- added SW4: SW_Push, Button_Switch_SMD:SW_SPST_KMR2, F.Cu at (272.9, 94.4)
- added SW5: SW_Push, Button_Switch_SMD:SW_SPST_KMR2, F.Cu at (134.1, 105.1)
- added SW6: SW_Push, Button_Switch_SMD:SW_SPST_KMR2, F.Cu at (128.1, 105.0)
- C1: value 22uF 50V -> 10uF 35V; footprint Capacitor_SMD:CP_Elec_5x5.8 -> Capacitor_SMD:C_1210_3225Metric_Pad1.42x2.65mm_HandSolder
- C10: value 0.22uF 25V -> 0.1uF; footprint Capacitor_SMD:C_0603_1608Metric_Pad1.05x0.95mm_HandSolder -> Capacitor_SMD:C_0603_1608Metric
- C11: value 0.1uF 50V -> 0.1uF; footprint Capacitor_SMD:C_0805_2012Metric_Pad1.15x1.40mm_HandSolder -> Capacitor_SMD:C_0603_1608Metric
- C12: value 0.01uF -> 0.47uF 16V; footprint Capacitor_SMD:C_0603_1608Metric_Pad1.05x0.95mm_HandSolder -> Capacitor_SMD:C_0603_1608Metric
- C13: value 82uF -> 0.47uF 6.3V; footprint Capacitor_SMD:CP_Elec_6.3x5.8 -> Capacitor_SMD:C_0603_1608Metric
- C14: value 330uF -> 0.1uF 50V; footprint Capacitor_SMD:CP_Elec_6.3x7.7 -> Capacitor_SMD:C_0603_1608Metric
- C2: value 220uF 25V -> 4.7uF 6.3V; footprint Capacitor_THT:CP_Radial_D6.3mm_P2.50mm -> Capacitor_SMD:C_0805_2012Metric_Pad1.15x1.40mm_HandSolder
- C3: value 0.01uF -> 100uF; footprint Capacitor_SMD:C_0603_1608Metric_Pad1.05x0.95mm_HandSolder -> Capacitor_THT:CP_Radial_D6.3mm_P2.50mm
- C4: value 82uF -> 0.1uF; footprint Capacitor_SMD:CP_Elec_6.3x5.8 -> Capacitor_SMD:C_0603_1608Metric
- C5: value 330uF -> 0.1uF; footprint Capacitor_SMD:CP_Elec_6.3x7.7 -> Capacitor_SMD:C_0603_1608Metric
- C6: value 0.1uF -> 0.47uF 16V; footprint Capacitor_SMD:C_0805_2012Metric_Pad1.15x1.40mm_HandSolder -> Capacitor_SMD:C_0603_1608Metric
- C7: value 0.1uF 50V -> 0.47uF 6.3V; footprint Capacitor_SMD:C_0805_2012Metric_Pad1.15x1.40mm_HandSolder -> Capacitor_SMD:C_0603_1608Metric
- C8: footprint Capacitor_SMD:C_0805_2012Metric_Pad1.15x1.40mm_HandSolder -> Capacitor_SMD:C_0603_1608Metric
- C9: footprint Capacitor_SMD:CP_Elec_8x10.5 -> Capacitor_THT:CP_Radial_D6.3mm_P2.50mm
- D1: footprint PTVS3V3P1UP:SOD128 -> Diode_THT:D_DO-201AD_P3.81mm_Vertical_AnodeUp
- D2: value SL04-E3-08 -> GREEN; footprint Diode_SMD:D_SOD-123F -> LED_SMD:LED_0603_1608Metric_Castellated
- D3: value B330 -> RED; footprint Diode_SMD:D_SMA -> LED_SMD:LED_0603_1608Metric_Castellated
- D4: value GREEN -> RED; footprint LED_SMD:LED_0603_1608Metric_Pad1.05x0.95mm_HandSolder -> LED_SMD:LED_0603_1608Metric_Castellated
- J1: footprint TerminalBlock:TerminalBlock_bornier-2_P5.08mm -> TerminalBlock_Phoenix:TerminalBlock_Phoenix_MKDS-1,5-2-5.08_1x02_P5.08mm_Horizontal
- J5: value TerminalBlock_02x04 -> Screw_Terminal_01x04; footprint mylib:DG500B-5.0-4P14 -> TerminalBlock_Phoenix:TerminalBlock_Phoenix_MKDS-1,5-4-5.08_1x04_P5.08mm_Horizontal
- Q1, Q2, Q5, Q6: footprint Package_TO_SOT_SMD:SOT-23_Handsoldering -> Package_TO_SOT_SMD:SOT-23
- Q10, Q11, Q12, Q14, Q15, Q16: footprint Package_TO_SOT_SMD:SuperSOT-3 -> Package_TO_SOT_SMD:SOT-23
- Q13, Q9: value 2N7002 -> FDV304; footprint Package_TO_SOT_SMD:SOT-23_Handsoldering -> Package_TO_SOT_SMD:SOT-23
- Q3, Q4, Q7, Q8: value BC327 -> Q_PMOS_GSD; footprint Package_TO_SOT_THT:TO-92_Inline -> Package_TO_SOT_SMD:SOT-23
- R1, R11, R12, R2: value 4.7k -> 1k; footprint Resistor_SMD:R_0603_1608Metric_Pad1.05x0.95mm_HandSolder -> Resistor_SMD:R_0603_1608Metric
- R10, R17, R18, R19, R20, R7, R8, R9: value 100k -> 10k; footprint Resistor_SMD:R_0603_1608Metric_Pad1.05x0.95mm_HandSolder -> Resistor_SMD:R_0603_1608Metric
- R13, R14, R3, R4: value 47k -> 10k; footprint Resistor_SMD:R_0603_1608Metric_Pad1.05x0.95mm_HandSolder -> Resistor_SMD:R_0603_1608Metric
- R15, R16, R5, R6: footprint Resistor_SMD:R_0805_2012Metric_Pad1.15x1.40mm_HandSolder -> Resistor_SMD:R_0603_1608Metric
- R21: value 47.5k -> 0.33; footprint Resistor_SMD:R_0603_1608Metric_Pad1.05x0.95mm_HandSolder -> Resistor_SMD:R_2512_6332Metric
- R22: value 2k -> 1M; footprint Resistor_SMD:R_0603_1608Metric_Pad1.05x0.95mm_HandSolder -> Resistor_SMD:R_0603_1608Metric
- R23: value 10k -> 1k; footprint Resistor_SMD:R_0603_1608Metric_Pad1.05x0.95mm_HandSolder -> Resistor_SMD:R_0603_1608Metric
- R24: value 4.7k -> 10k; footprint Resistor_SMD:R_0603_1608Metric_Pad1.05x0.95mm_HandSolder -> Resistor_SMD:R_0603_1608Metric
- R25, R40: value 10k -> 220; footprint Resistor_SMD:R_0603_1608Metric_Pad1.05x0.95mm_HandSolder -> Resistor_SMD:R_0603_1608Metric
- R26: value 110 -> 0.33; footprint Resistor_SMD:R_0603_1608Metric_Pad1.05x0.95mm_HandSolder -> Resistor_SMD:R_2512_6332Metric; moved to B.Cu
- R27: value 5k -> 1M; footprint Resistor_SMD:R_0603_1608Metric_Pad1.05x0.95mm_HandSolder -> Resistor_SMD:R_0603_1608Metric
- R28: value 220 -> 1k; footprint Resistor_SMD:R_0603_1608Metric_Pad1.05x0.95mm_HandSolder -> Resistor_SMD:R_0603_1608Metric
- R29, R30, R31, R32, R33, R34, R35, R36, R37, R46, R47, R48, R49, R50, R51, R52, R53, R54: footprint Resistor_SMD:R_0603_1608Metric_Pad1.05x0.95mm_HandSolder -> Resistor_SMD:R_0603_1608Metric
- R38: value 47.5k -> 10k; footprint Resistor_SMD:R_0603_1608Metric_Pad1.05x0.95mm_HandSolder -> Resistor_SMD:R_0603_1608Metric
- R39: value 2k -> 220; footprint Resistor_SMD:R_0603_1608Metric_Pad1.05x0.95mm_HandSolder -> Resistor_SMD:R_0603_1608Metric
- R41: value 4.7k -> 33k; footprint Resistor_SMD:R_0603_1608Metric_Pad1.05x0.95mm_HandSolder -> Resistor_SMD:R_0603_1608Metric
- R42: value 10k -> 33k; footprint Resistor_SMD:R_0603_1608Metric_Pad1.05x0.95mm_HandSolder -> Resistor_SMD:R_0603_1608Metric
- RV1, RV10: value 50k -> 5k; footprint Potentiometer_THT:Potentiometer_Vishay_T73XX_Horizontal -> Potentiometer_THT:Potentiometer_Bourns_3266W_Vertical
- U1: value LM2574M-3.3 -> L78L33_SOT89; footprint Package_SO:SOIC-14W_7.5x9.0mm_P1.27mm -> Package_TO_SOT_SMD:SOT-89-3_Handsoldering
- U2: value A8498 -> DRV8840; footprint Package_SO:SOIC-8-1EP_3.9x4.9mm_P1.27mm_EP2.35x2.35mm -> SOP65P640X110-29N:SOP65P640X110-29N
- U3: value A3950SLP-T -> DRV8840; footprint Package_SO:HTSSOP-16-1EP_4.4x5mm_P0.65mm_EP3.4x5mm_Mask3x3mm_ThermalVias -> SOP65P640X110-29N:SOP65P640X110-29N
- moved Q16 239.2 mm to (127.9, 111.8), turned to 180 degrees
- moved R53 235.1 mm to (128.1, 114.5), turned to 180 degrees
- moved Q15 234.5 mm to (133.6, 111.8), turned to 180 degrees
- moved R54 231.9 mm to (128.1, 109.0), turned to 180 degrees
- moved Q13 231.2 mm to (136.5, 96.0), turned to 90 degrees
- moved RV10 231.0 mm to (126.9, 91.4), turned to 90 degrees
- moved R51 230.8 mm to (133.9, 109.0), turned to 180 degrees
- moved R40 228.6 mm to (116.1, 97.1)
- moved C14 225.8 mm to (141.8, 85.6), turned to 90 degrees
- moved R52 224.4 mm to (130.8, 113.6), turned to 270 degrees
- moved Q14 224.3 mm to (139.2, 111.8), turned to 180 degrees
- moved R38 224.1 mm to (140.1, 97.0)
- moved R49 223.6 mm to (136.4, 113.5), turned to 270 degrees
- moved R50 221.0 mm to (133.9, 114.6), turned to 180 degrees
- moved R48 220.5 mm to (139.4, 109.0), turned to 180 degrees
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Connections:
- C1 pad 1: /Motor1 supply/24V -> /Power section/24V
- C10 pad 1: GND -> /Power section/24V
- C10 pad 2: Net-(C10-Pad2) -> GND
- C11 pad 1: Net-(C11-Pad1) -> /Power section/24V
- C11 pad 2: Net-(C11-Pad2) -> GND
- C12 pad 2: Net-(C12-Pad2) -> /Power section/24V
- C13 pad 1: /Motor1 supply/24V -> Net-(C13-Pad1)
- C14 pad 1: /Motor2 driver/VBB -> Net-(C14-Pad1)
- C14 pad 2: GND -> Net-(C14-Pad2)
- C3 pad 1: Net-(C3-Pad1) -> /Power section/24V
- C3 pad 2: Net-(C3-Pad2) -> GND
- C4 pad 1: /Motor1 supply/24V -> /Power section/24V
- C5 pad 1: /Motor1 driver/VBB -> /Power section/24V
- C6 pad 1: GND -> Net-(C6-Pad1)
- C6 pad 2: /Motor1 supply/24V -> /Power section/24V
- C7 pad 1: /Motor1 driver/VBB -> Net-(C7-Pad1)
- C8 pad 1: /Motor1 driver/VBB -> Net-(C8-Pad1)
- C9 pad 1: /Motor1 driver/VBB -> /Power section/24V
- D1 pad 1: /Motor1 supply/24V -> /Power section/24V
- D2 pad 1: Net-(D2-Pad1) -> GND
- D2 pad 2: GND -> Net-(D2-Pad2)
- D3 pad 1: Net-(C3-Pad2) -> GND
- D3 pad 2: GND -> Net-(D3-Pad2)
- D4 pad 1: Net-(D4-Pad1) -> GND
- J1 pad 1: GND -> /Power section/VIN
- J1 pad 2: /Power section/VIN -> GND
- J11 pad 1: /Motor2 driver/OUTA -> /Motor2 driver/OUT1
- J11 pad 2: /Motor2 driver/OUTB -> /Motor2 driver/OUT2
- J5 pad 1: GND -> /ttl-to-plc/OUT1
- J5 pad 2: /ttl-to-plc/OUT4 -> /ttl-to-plc/OUT2
- J5 pad 3: GND -> /ttl-to-plc/OUT3
- J5 pad 4: /ttl-to-plc/OUT3 -> /ttl-to-plc/OUT4
- J6 pad 3: /Motor1 driver/MODE -> /Motor1 driver/DECAY
- J7 pad 1: /Motor2 driver/MODE -> /Motor2 driver/ENABLE
- J7 pad 3: /Motor2 driver/ENABLE -> /Motor2 driver/DECAY
- J9 pad 1: /Motor1 driver/OUTA -> /Motor1 driver/OUT2
- J9 pad 2: /Motor1 driver/OUTB -> /Motor1 driver/OUT1
- Q12 pad 2: /Motor1 driver/MODE -> /Motor1 driver/DECAY
- Q13 pad 2: GND -> /Motor1 3V3 <- PLC/3V3
- Q13 pad 3: Net-(D7-Pad1) -> Net-(Q13-Pad3)
- Q14 pad 2: /Motor2 driver/MODE -> /Motor2 driver/ENABLE
- Q16 pad 2: /Motor2 driver/ENABLE -> /Motor2 driver/DECAY
- Q3 pad 1: /ttl-to-plc/OUT1 -> Net-(Q3-Pad1)
- Q3 pad 2: Net-(Q3-Pad2) -> /ttl-to-plc/OUT1
- Q3 pad 3: /Motor1 supply/24V -> /Power section/24V
- Q4 pad 1: /ttl-to-plc/OUT3 -> Net-(Q4-Pad1)
- Q4 pad 2: Net-(Q4-Pad2) -> /ttl-to-plc/OUT3
- Q4 pad 3: /Motor1 supply/24V -> /Power section/24V
- Q7 pad 1: /ttl-to-plc/OUT2 -> Net-(Q7-Pad1)
- Q7 pad 2: Net-(Q7-Pad2) -> /ttl-to-plc/OUT2
- Q7 pad 3: /Motor1 supply/24V -> /Power section/24V
- Q8 pad 1: /ttl-to-plc/OUT4 -> Net-(Q8-Pad1)
- Q8 pad 2: Net-(Q8-Pad2) -> /ttl-to-plc/OUT4
- Q8 pad 3: /Motor1 supply/24V -> /Power section/24V
- Q9 pad 2: GND -> /Motor1 3V3 <- PLC/3V3
- Q9 pad 3: Net-(D4-Pad1) -> Net-(Q9-Pad3)
- R15 pad 2: Net-(Q7-Pad2) -> Net-(Q7-Pad1)
- R16 pad 2: Net-(Q8-Pad2) -> Net-(Q8-Pad1)
- R17 pad 1: Net-(Q7-Pad2) -> Net-(Q7-Pad1)
- R17 pad 2: /Motor1 supply/24V -> /Power section/24V
- R18 pad 1: Net-(Q8-Pad2) -> Net-(Q8-Pad1)
- R18 pad 2: /Motor1 supply/24V -> /Power section/24V
- R22 pad 1: GND -> Net-(C6-Pad1)
- R22 pad 2: Net-(R22-Pad2) -> /Power section/24V
- R23 pad 1: /Motor1 driver/VBB -> Net-(Q9-Pad1)
- R24 pad 1: Net-(Q9-Pad1) -> /Motor1 3V3 <- PLC/3V3
- R24 pad 2: /Motor1 driver/VBB -> Net-(Q9-Pad1)
- R25 pad 1: Net-(Q9-Pad1) -> Net-(Q9-Pad3)
- R25 pad 2: GND -> Net-(D3-Pad2)
- R26 pad 1: /Motor1 3V3 <- PLC/3V3 -> Net-(R26-Pad1)
- R26 pad 2: Net-(D4-Pad2) -> GND
- R27 pad 1: /Motor1 3V3 <- PLC/3V3 -> Net-(C12-Pad1)
- R27 pad 2: Net-(R27-Pad2) -> /Power section/24V
- R28 pad 1: Net-(D5-Pad1) -> Net-(Q13-Pad1)
- R37 pad 1: /Motor1 driver/MODE -> /Motor1 driver/DECAY
- R38 pad 1: Net-(R38-Pad1) -> /Motor1 3V3 <- PLC/3V3
- R38 pad 2: GND -> Net-(Q13-Pad1)
- R39 pad 1: GND -> Net-(Q13-Pad3)
- R39 pad 2: Net-(R39-Pad2) -> Net-(D4-Pad2)
- R40 pad 1: /Motor2 driver/VBB -> /Motor1 3V3 <- PLC/3V3
- R40 pad 2: Net-(R40-Pad2) -> Net-(D2-Pad2)
- R41 pad 1: Net-(Q13-Pad1) -> /Motor1 3V3 <- PLC/3V3
- R41 pad 2: /Motor2 driver/VBB -> /Motor1 driver/DECAY
- R42 pad 1: Net-(Q13-Pad1) -> /Motor1 3V3 <- PLC/3V3
- R42 pad 2: GND -> /Motor2 driver/DECAY
- R48 pad 1: /Motor2 driver/MODE -> /Motor2 driver/ENABLE
- R5 pad 2: Net-(Q3-Pad2) -> Net-(Q3-Pad1)
- R54 pad 1: /Motor2 driver/ENABLE -> /Motor2 driver/DECAY
- R6 pad 2: Net-(Q4-Pad2) -> Net-(Q4-Pad1)
- R7 pad 1: Net-(Q3-Pad2) -> Net-(Q3-Pad1)
- R7 pad 2: /Motor1 supply/24V -> /Power section/24V
- R8 pad 1: Net-(Q4-Pad2) -> Net-(Q4-Pad1)
- R8 pad 2: /Motor1 supply/24V -> /Power section/24V
- RV1 pad 1: Net-(RV1-Pad1) -> GND
- RV1 pad 2: Net-(R23-Pad2) -> Net-(RV1-Pad2)
- RV1 pad 3: Net-(R22-Pad2) -> Net-(C7-Pad1)
- RV10 pad 1: Net-(RV10-Pad1) -> GND
- RV10 pad 2: Net-(R40-Pad2) -> Net-(RV10-Pad2)
- RV10 pad 3: Net-(R39-Pad2) -> Net-(C13-Pad1)
- U1 pad 1: (no net) -> /Motor1 3V3 <- PLC/3V3
- U1 pad 2: (no net) -> GND
- U1 pad 3: /Motor1 3V3 <- PLC/3V3 -> /Power section/24V
- U2 pad 1: Net-(C3-Pad1) -> Net-(C8-Pad1)
- U2 pad 2: GND -> Net-(C8-Pad2)
- U2 pad 3: Net-(R21-Pad1) -> Net-(C6-Pad1)
- U2 pad 4: GND -> /Power section/24V
- U2 pad 5: Net-(R22-Pad2) -> /Motor1 driver/OUT1
- U2 pad 6: /Motor1 driver/VBB -> Net-(R21-Pad1)
- U2 pad 7: Net-(C3-Pad2) -> /Motor1 driver/OUT2
- U2 pad 8: /Motor1 supply/24V -> /Motor1 driver/OUT2
- U2 pad 9: GND -> Net-(R21-Pad1)
- U3 pad 1: Net-(R28-Pad2) -> Net-(C14-Pad1)
- U3 pad 10: /Motor1 driver/OUTB -> /Motor2 driver/OUT1
- U3 pad 11: Net-(C11-Pad1) -> /Power section/24V
- U3 pad 12: Net-(C11-Pad2) -> Net-(RV10-Pad2)
- U3 pad 13: GND -> Net-(RV10-Pad2)
- U3 pad 14: Net-(C8-Pad2) -> GND
- U3 pad 15: Net-(C10-Pad2) -> Net-(C13-Pad1)
- U3 pad 16: Net-(U3-Pad16) -> /Motor1 3V3 <- PLC/3V3
- U3 pad 17: GND -> /Motor1 3V3 <- PLC/3V3
- U3 pad 2: /Motor1 driver/MODE -> Net-(C14-Pad2)
- U3 pad 3: /Motor1 3V3 <- PLC/OUT2 -> Net-(C12-Pad1)
- U3 pad 4: GND -> /Power section/24V
- U3 pad 5: Net-(R27-Pad2) -> /Motor2 driver/OUT1
- U3 pad 6: /Motor1 driver/ENABLE -> Net-(R26-Pad1)
- U3 pad 7: /Motor1 driver/OUTA -> /Motor2 driver/OUT2
- U3 pad 8: GND -> /Motor2 driver/OUT2
- U3 pad 9: /Motor1 driver/VBB -> Net-(R26-Pad1)
Routing:
- net /Power section/24V: track 0.00 -> 34.8 mm, vias 0 -> 12
- net /Motor2 driver/OUT1: track 0.00 -> 23.8 mm, vias 0 -> 12
- net Net-(D2-Pad1): track 18.8 -> 0.00 mm
- net /Motor2 driver/OUT2: track 0.00 -> 18.6 mm
- net Net-(RV10-Pad2): track 0.00 -> 14.1 mm, vias 0 -> 2
- net /Motor2 driver/DECAY: track 0.00 -> 9.17 mm, vias 0 -> 1
- net /Motor2 driver/ENABLE: track 0.00 -> 8.97 mm, vias 0 -> 1
- net Net-(C13-Pad1): track 0.00 -> 8.71 mm
- net Net-(R26-Pad1): track 0.00 -> 8.59 mm, vias 0 -> 10
- net /Motor2 3V3 <- PLC/OUT2: track 0.00 -> 8.41 mm, vias 0 -> 1
- net Net-(Q4-Pad2): track 7.92 -> 0.00 mm
- net Net-(Q8-Pad2): track 7.81 -> 0.00 mm
- net Net-(Q7-Pad2): track 7.71 -> 0.00 mm
- net Net-(Q3-Pad2): track 7.61 -> 0.00 mm
- net Net-(C12-Pad1): track 0.00 -> 5.12 mm
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- added copper zone on B.Cu, net /Motor2 driver/OUT1
- added copper zone on F.Cu, net /Motor2 driver/OUT1
- added copper zone on F.Cu, net /Power section/24V
- added copper zone on B.Cu, net Net-(R26-Pad1)
Other:
- net class Default: clearance 0.254 -> 0.1; trace_width 0.25 -> 0.45; via_dia 0.8 -> 0.45; via_drill 0.4 -> 0.2
- rule trace_clearance: 0.254 -> 0.1
- rule via_min_drill: 0.3 -> 0.2
- rule via_min_size: 0.4 -> 0.45
