File: power-section.sch (KiCad schematic (older format))
At the start: 6 parts, among them U1 L78L33_SOT89

Commit message: Added switch for selecting Low/High power motor. Added thermal pads around motor controllers.
Parts:
- D1: footprint Diode_THT:D_DO-201AD_P3.81mm_Vertical_KathodeUp -> Diode_THT:D_DO-201AD_P5.08mm_Vertical_KathodeUp
Changed lines of the file:
@@
 F 0 "D1" H 4750 1650 50  0000 L CNN
 F 1 "SB530" H 4650 1750 50  0000 L CNN
-F 2 "Diode_THT:D_DO-201AD_P3.81mm_Vertical_KathodeUp" H 4800 1850 50  0001 C CNN
+F 2 "Diode_THT:D_DO-201AD_P5.08mm_Vertical_KathodeUp" H 4800 1850 50  0001 C CNN
 F 3 "~" H 4800 1850 50  0001 C CNN
 	1    4800 1850
